Commit message: Update

File: marrtinorobot2/marrtinorobot2_description/urdf/yellow_properties.urdf.xacro (robot description, xacro)
@@ -1,7 +1,7 @@
 <?xml version="1.0"?>
 <robot xmlns:xacro="http://ros.org/wiki/xacro">
-  <xacro:property name="base_length" value="0.23" />
-  <xacro:property name="base_width" value="0.17" />
-  <xacro:property name="base_height" value="0.12" />
+  <xacro:property name="base_length" value="0.33" />
+  <xacro:property name="base_width" value="0.19" />
+  <xacro:property name="base_height" value="0.115" />
   <xacro:property name="base_mass" value="1" />
   <xacro:property name="wheel_radius" value="0.0725" />
