Commit message: Update docker

File: marrtinorobot2/marrtinorobot2_description/urdf/2wd_properties.urdf.xacro (robot description, xacro)
@@ -1,7 +1,7 @@
 <?xml version="1.0"?>
 <robot xmlns:xacro="http://ros.org/wiki/xacro">
-  <xacro:property name="base_length" value="0.30" />
-  <xacro:property name="base_width" value="0.26" />
-  <xacro:property name="base_height" value="0.08" />
+  <xacro:property name="base_length" value="0.34" />
+  <xacro:property name="base_width" value="0.29" />
+  <xacro:property name="base_height" value="0.09" />
   <xacro:property name="base_mass" value="1" />
   <xacro:property name="wheel_radius" value="0.07" />
@@ -15,8 +15,8 @@
   <xacro:property name="rear_caster_wheel" value="true" />
   <xacro:property name="laser_pose">
-    <origin xyz="0.10 0 0.10" rpy="0 0 0"/>
+    <origin xyz="0 0 0.10" rpy="0 0 0"/>
   </xacro:property>
   <xacro:property name="depth_sensor_pose">
-    <origin xyz="0.14 0.0 0.045" rpy="0 0 0"/>
+    <origin xyz="0.14 0.0 0.055" rpy="0 0 0"/>
   </xacro:property>
 </robot>

Commit message: Blockly

File: marrtinorobot2/marrtinorobot2_description/urdf/2wd_properties.urdf.xacro (robot description, xacro)
@@ -1,5 +1,5 @@
 <?xml version="1.0"?>
 <robot xmlns:xacro="http://ros.org/wiki/xacro">
-  <xacro:property name="base_length" value="0.34" />
+  <xacro:property name="base_length" value="0.28" />
   <xacro:property name="base_width" value="0.29" />
   <xacro:property name="base_height" value="0.09" />
