Commit message: Update mecanum

File: marrtinorobot2/marrtinorobot2_description/urdf/mecanum_properties.urdf.xacro (robot description, xacro)
@@ -1,11 +1,11 @@
 <?xml version="1.0"?>
 <robot xmlns:xacro="http://ros.org/wiki/xacro">
-  <xacro:property name="base_length" value="0.445" />
+  <xacro:property name="base_length" value="0.270" />
   <xacro:property name="base_width" value="0.200" />
-  <xacro:property name="base_height" value="0.129" />
+  <xacro:property name="base_height" value="0.100" />
   <xacro:property name="base_mass" value="10" />
-  <xacro:property name="wheel_radius" value="0.07162" />
-  <xacro:property name="wheel_width" value="0.05" />
-  <xacro:property name="wheel_pos_x" value="0.120" />
+  <xacro:property name="wheel_radius" value="0.0475" />
+  <xacro:property name="wheel_width" value="0.045" />
+  <xacro:property name="wheel_pos_x" value="0.075" />
   <xacro:property name="wheel_pos_y" value="0.1355" />
   <xacro:property name="wheel_pos_z" value="-0.04788" />
@@ -13,8 +13,8 @@
   <xacro:property name="wheel_torque" value="20" />
   <xacro:property name="laser_pose">
-    <origin xyz="-0.0475 0 0.125" rpy="0 0 0"/>
+    <origin xyz="0 0 0.125" rpy="0 0 0"/>
   </xacro:property>
   <xacro:property name="depth_sensor_pose">
-    <origin xyz="0.2375 0 0.06" rpy="0 0 0"/>
+    <origin xyz="0.18 0 0.06" rpy="0 0 0"/>
   </xacro:property>
 </robot>
